File: mushroomFarmKiCAD.kicad_pcb (KiCad board)
At the start: 2 copper layers, 22 parts, among them J1 Screw_Terminal_01x02, J2 RelayConn, J3 DHT22Conn, J4 ESP32pin, J5 ESP32pin, U1 L7812, U2 L7812, U3 L7806

Commit message: Created PCB added 3d models, improve pcb
Parts:
- J1: footprint TerminalBlock_Altech:Altech_AK300_1x02_P5.00mm_45-Degree -> TerminalBlock_Phoenix:TerminalBlock_Phoenix_MKDS-1,5-2_1x02_P5.00mm_Horizontal
- J2: footprint Connector_PinHeader_2.54mm:PinHeader_1x06_P2.54mm_Vertical -> Connector_PinSocket_2.54mm:PinSocket_1x06_P2.54mm_Vertical
- J3: footprint Connector_PinHeader_2.54mm:PinHeader_1x04_P2.54mm_Vertical -> Connector_PinSocket_2.54mm:PinSocket_1x04_P2.54mm_Vertical
- J4, J5: footprint Connector_PinHeader_2.54mm:PinHeader_1x15_P2.54mm_Vertical -> Connector_PinSocket_2.54mm:PinSocket_1x15_P2.54mm_Vertical
- moved J1 4.60 mm to (71.8, 93.0), turned to -90 degrees
Routing:
- net Net-(J1-Pad1): track 10.1 -> 29.9 mm
- net Net-(C2-Pad1): track 17.7 -> 20.3 mm
Other:
- board outline added: 150.9 x 67.6 mm
